File: hardware/booster-I-board/booster-I-board.kicad_pcb (KiCad board)
At the start: 2 copper layers, 100 x 100 mm, 3 parts, among them J1 7461057, J2 7461057

Commit message: ftdi board + random stuff
Parts:
- added J3: 3-647166-2, Library:36471662, F.Cu at (168.3, 50.5)
- added TH1: NTCGS163JF103FT8, Resistor_SMD:R_0603_1608Metric_Pad0.98x0.95mm_HandSolder, B.Cu at (161.6, 89.5)
Routing:
- net Net-(J3-Pin_2): track 0.00 -> 43.1 mm, vias 0 -> 1
- net Net-(J3-Pin_1): track 0.00 -> 42.2 mm, vias 0 -> 1
- added copper zone on F.Cu, net Net-(J1-Pad1)
- added copper zone on B.Cu, net Net-(J2-Pad1)
- removed copper zone on B.Cu, net Net-(J1-Pad1)
- removed copper zone on F.Cu, net Net-(J2-Pad1)
Other:
- board size 100 x 100 mm -> 101 x 101 mm
