File: hardware/booster-tc-driver/booster-tc-driver.kicad_pcb (KiCad board)
At the start: 4 copper layers, 53.3 x 72 mm, 146 parts, among them IC1 AD5160BRJZ5-RL7, IC2 AD5160BRJZ5-RL7, IC3 BD50FD0WHFP-TR, IC4 CAT4109V-GT2, IC5 L4940D2T12-TR, IC6 SI4564DY-T1-GE3, IC7 SI4564DY-T1-GE3, IC8 SI4564DY-T1-GE3, IC9 SI4564DY-T1-GE3, J1 62201021121, J10 3-647166-2, J2 EHT-105-01-S-D, J3 3-647166-2, J4 22-23-2021, J5 22-23-2021, J6 22-23-2021, J7 3-647166-2, J8 B4B-PH-SM4-TB, Q1 T2N7002AK, SW1 SW_SPDT, U1 STM32G474CBTx, U10 LT1963AxST-3.3, U2 AOZ1284PI, U3 CSTNE8M00G550000R0, U4 IF-D95T << must be T, U5 IF-E96E, U6 IF-D95T << must be T, U7 AOZ1284PI, U8 UCC21520DW, U9 UCC21520DW

Commit message: driver board work
Parts:
- added C64: .1uf 885012208087, Capacitor_SMD:C_1206_3216Metric_Pad1.33x1.80mm_HandSolder, B.Cu at (22.7, 22.9)
- added C65: .1uf 885012208087, Capacitor_SMD:C_1206_3216Metric_Pad1.33x1.80mm_HandSolder, B.Cu at (21.4, 29.4)
- added C66: .1uf 885012208087, Capacitor_SMD:C_1206_3216Metric_Pad1.33x1.80mm_HandSolder, B.Cu at (22.2, 19.0)
- added C67: 2u2 C3225X7R1H225K250AB, Capacitor_SMD:C_1210_3225Metric_Pad1.33x2.70mm_HandSolder, B.Cu at (28.8, 24.0)
- added C68: 2u2 C3225X7R1H225K250AB, Capacitor_SMD:C_1210_3225Metric_Pad1.33x2.70mm_HandSolder, B.Cu at (32.2, 24.0)
- added C69: 2u2 C3225X7R1H225K250AB, Capacitor_SMD:C_1210_3225Metric_Pad1.33x2.70mm_HandSolder, B.Cu at (28.8, 18.8)
- added C70: 2u2 C3225X7R1H225K250AB, Capacitor_SMD:C_1210_3225Metric_Pad1.33x2.70mm_HandSolder, B.Cu at (32.2, 18.8)
- added C71: .1uf 885012208087, Capacitor_SMD:C_1206_3216Metric_Pad1.33x1.80mm_HandSolder, B.Cu at (51.8, 27.0)
- added C72: 2u2 C3225X7R1H225K250AB, Capacitor_SMD:C_1210_3225Metric_Pad1.33x2.70mm_HandSolder, B.Cu at (32.8, 29.2)
- added C73: .1uf 885012208087, Capacitor_SMD:C_1206_3216Metric_Pad1.33x1.80mm_HandSolder, B.Cu at (35.6, 30.6)
- added C74: .1uf 885012208087, Capacitor_SMD:C_1206_3216Metric_Pad1.33x1.80mm_HandSolder, B.Cu at (54.2, 27.0)
- added C75: 2u2 C3225X7R1H225K250AB, Capacitor_SMD:C_1210_3225Metric_Pad1.33x2.70mm_HandSolder, B.Cu at (63.2, 20.3)
- added C76: 2u2 C3225X7R1H225K250AB, Capacitor_SMD:C_1210_3225Metric_Pad1.33x2.70mm_HandSolder, B.Cu at (59.8, 20.3)
- added C77: 2u2 C3225X7R1H225K250AB, Capacitor_SMD:C_1210_3225Metric_Pad1.33x2.70mm_HandSolder, B.Cu at (63.2, 25.5)
- added C78: 2u2 C3225X7R1H225K250AB, Capacitor_SMD:C_1210_3225Metric_Pad1.33x2.70mm_HandSolder, B.Cu at (59.7, 25.5)
- added C79: 2u2 C3225X7R1H225K250AB, Capacitor_SMD:C_1210_3225Metric_Pad1.33x2.70mm_HandSolder, B.Cu at (49.3, 37.5)
- added C80: .1uf C0603C104K3RECTU, Capacitor_SMD:C_0603_1608Metric_Pad1.08x0.95mm_HandSolder, B.Cu at (46.6, 36.2)
- added C81: .1uf C0603C104K3RECTU, Capacitor_SMD:C_0603_1608Metric_Pad1.08x0.95mm_HandSolder, B.Cu at (45.0, 40.6)
- added C82: .1uf C0603C104K3RECTU, Capacitor_SMD:C_0603_1608Metric_Pad1.08x0.95mm_HandSolder, B.Cu at (44.4, 36.2)
- added C83: 2u2 C3225X7R1H225K250AB, Capacitor_SMD:C_1210_3225Metric_Pad1.33x2.70mm_HandSolder, B.Cu at (59.7, 30.8)
- added C84: 2u2 C3225X7R1H225K250AB, Capacitor_SMD:C_1210_3225Metric_Pad1.33x2.70mm_HandSolder, B.Cu at (63.2, 30.8)
- added C85: 2u2 C3225X7R1H225K250AB, Capacitor_SMD:C_1210_3225Metric_Pad1.33x2.70mm_HandSolder, B.Cu at (34.9, 72.4)
- added C86: 2u2 C3225X7R1H225K250AB, Capacitor_SMD:C_1210_3225Metric_Pad1.33x2.70mm_HandSolder, B.Cu at (39.2, 76.6)
- added C87: 2u2 C3225X7R1H225K250AB, Capacitor_SMD:C_1210_3225Metric_Pad1.33x2.70mm_HandSolder, B.Cu at (39.2, 79.9)
- added C88: 2u2 C3225X7R1H225K250AB, Capacitor_SMD:C_1210_3225Metric_Pad1.33x2.70mm_HandSolder, B.Cu at (27.0, 78.5)
- added C89: 2u2 C3225X7R1H225K250AB, Capacitor_SMD:C_1210_3225Metric_Pad1.33x2.70mm_HandSolder, B.Cu at (27.0, 74.7)
- added C90: .1uf 885012208087, Capacitor_SMD:C_1206_3216Metric_Pad1.33x1.80mm_HandSolder, B.Cu at (46.4, 73.4)
- added C91: .1uf 885012208087, Capacitor_SMD:C_1206_3216Metric_Pad1.33x1.80mm_HandSolder, B.Cu at (39.3, 72.4)
- added C92: .1uf 885012208087, Capacitor_SMD:C_1206_3216Metric_Pad1.33x1.80mm_HandSolder, B.Cu at (28.9, 85.4)
- added C93: .1uf 885012208087, Capacitor_SMD:C_1206_3216Metric_Pad1.33x1.80mm_HandSolder, B.Cu at (26.4, 85.4)
- added C94: .1uf 885012208087, Capacitor_SMD:C_1206_3216Metric_Pad1.33x1.80mm_HandSolder, B.Cu at (23.9, 85.4)
- added C95: .1uf 885012208087, Capacitor_SMD:C_1206_3216Metric_Pad1.33x1.80mm_HandSolder, B.Cu at (21.4, 85.4)
- C15, Q1, R3, R4, R5: moved to B.Cu
- C35: value .1uf 885012208087 -> .1uf C0603C104K3RECTU; footprint Capacitor_SMD:C_1206_3216Metric_Pad1.33x1.80mm_HandSolder -> Capacitor_SMD:C_0603_1608Metric_Pad1.08x0.95mm_HandSolder
- IC4: moved to F.Cu
- moved C7 17.9 mm to (61.7, 73.7), turned to 0 degrees
- moved IC4 11.9 mm to (45.9, 72.5), turned to -90 degrees
- moved Q1 11.1 mm to (62.4, 85.7)
- moved R26 10.6 mm to (42.9, 73.1), turned to 90 degrees
- moved R27 10.4 mm to (41.4, 73.1), turned to 90 degrees
- moved R9 10.2 mm to (55.1, 75.9), turned to 180 degrees
- moved R7 9.97 mm to (52.7, 73.6), turned to 180 degrees
- moved R3 9.06 mm to (40.1, 84.2), turned to -90 degrees
- moved D10 7.77 mm to (50.5, 79.5), turned to 90 degrees
- moved R5 7.65 mm to (59.4, 85.6)
- moved U5 7.63 mm to (58.1, 88.0)
- moved R4 7.63 mm to (58.6, 82.2)
- moved C15 6.53 mm to (49.5, 85.4)
- moved C34 6.28 mm to (52.9, 74.1)
- moved R25 5.64 mm to (44.4, 73.1), turned to 90 degrees
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Connections:
- C35 pad 1: VDDA -> GND
- C35 pad 2: GND -> VDDA
Routing:
- net GND: track 254.8 -> 357.9 mm, vias 105 -> 106
- net VDD: track 24.5 -> 56.0 mm, vias 17 -> 21
- net +12V: track 125.4 -> 148.8 mm
- net Net-(IC4-LED3): track 3.62 -> 23.8 mm
- net Net-(IC4-LED2): track 3.81 -> 23.5 mm
- net Net-(IC4-LED1): track 4.34 -> 21.1 mm
- net /LED_VBUS: track 23.9 -> 7.67 mm, vias 1 -> 0
- net /LED_TMP: track 22.4 -> 9.28 mm, vias 1 -> 0
- net +5V: track 245.7 -> 234.1 mm, vias 6 -> 5
- net +24V: track 34.8 -> 44.5 mm, vias 9 -> 19
- net /LED_I_IN: track 20.0 -> 11.2 mm, vias 1 -> 0
- net /USART_RX: track 34.2 -> 42.1 mm
- net /VAC_IN: track 89.1 -> 96.4 mm
- net /MODE_IN: track 66.6 -> 73.3 mm
- net /VAC_SENSE: track 30.8 -> 24.5 mm
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Other:
- board text added: "BOOSTER DRIVER V1"
- board text added: "CT"
- board text added: "D13"
- board text added: "FAN"
- board text added: "PMP"
- board text added: "THERM"

Commit message: silkscreen + software cleanup
Parts:
- C3, C43, C45: value 330u 860020575013 -> 470u 860020474014; footprint Library:860020575013 -> Library:CAPPRD350W52D800H1300
- C72: value 2u2 C3225X7R1H225K250AB -> .1uf 885012208087; footprint Capacitor_SMD:C_1210_3225Metric_Pad1.33x2.70mm_HandSolder -> Capacitor_SMD:C_1206_3216Metric_Pad1.33x1.80mm_HandSolder
- C85: moved to F.Cu
- moved C85 41.7 mm to (39.3, 30.9), turned to 90 degrees
- moved C73 3.55 mm to (33.7, 27.6), turned to 0 degrees
- moved C72 1.92 mm to (33.7, 30.9), turned to 0 degrees
- moved C45 1.66 mm to (26.5, 27.9), turned to 90 degrees
- moved R10 1.08 mm to (33.4, 39.1)
- moved C12 0.71 mm to (61.5, 62.3)
- moved C43 0.68 mm to (33.3, 32.8), turned to 90 degrees
- moved C3 0.65 mm to (33.1, 71.0)
- moved C25 0.15 mm to (33.5, 64.4)
- moved C67 0.10 mm to (28.8, 23.9)
- moved C68 0.10 mm to (32.2, 23.9)
- moved C69 0.10 mm to (28.8, 18.7)
- moved C70 0.10 mm to (32.2, 18.7)
Connections:
- C85 pad 1: VDD -> VDRIVE
- U1 pad 18: /INT -> /SCR
- U1 pad 34: /SCR -> /INT
Routing:
- net /INT: track 41.2 -> 52.6 mm, vias 0 -> 2
- net GND: track 357.9 -> 350.7 mm, vias 106 -> 111
- net VDRIVE: track 98.6 -> 92.3 mm
- net +12V: track 148.8 -> 152.4 mm
- net /CT-: track 49.7 -> 47.7 mm
- net /I_PRI: track 31.5 -> 33.5 mm
- net /CS_DRIVE: track 144.6 -> 142.7 mm
- net /CT+: track 51.0 -> 49.1 mm
- net /I_L_IN: track 39.8 -> 38.2 mm
- net /PFC: track 104.1 -> 102.5 mm
- net /SPI_MOSI: track 168.7 -> 167.3 mm
- net /VAC_IN: track 96.4 -> 95.2 mm
- net VDD: track 56.0 -> 54.9 mm
- net /VREF: track 14.7 -> 13.7 mm
- net /THERM2: track 33.3 -> 32.4 mm
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
Commit message: schematic cleanup
Parts:
- L4, L5: value 22u 7443551221 -> 22u SRP7028A-220M; footprint Library:7443551221 -> Library:INDPM7366X300N
- moved L4 4.38 mm to (51.6, 55.2)
- moved L5 2.87 mm to (36.5, 39.1)
- moved C65 0.10 mm to (21.3, 29.4)
- moved C66 0.10 mm to (22.1, 19.0)
Connections:
- net /CS_DRIVE renamed CS_DRIVE
- net /CS_FAN renamed CS_FAN
- net /CT+ renamed CT+
- net /CT- renamed CT-
- net /DRIVE_EN renamed DRIVE_EN
- net /FAN_EN renamed FAN_EN
- net /Gate Drive Out/GDT1_A renamed GDT1_A
- net /Gate Drive Out/GDT1_B renamed GDT1_B
- net /Gate Drive Out/GDT2_A renamed GDT2_A
- net /Gate Drive Out/GDT2_B renamed GDT2_B
- net /INT renamed INT
- net /I_L renamed I_L
- net /I_L_IN renamed Net-(J2-Pad01)
- net /I_PRI renamed I_PRI
- net /LED_I_IN renamed LED_I_IN
- net /LED_TMP renamed LED_TMP
- net /LED_VBUS renamed LED_VBUS
- net /MODE_IN renamed MODE_IN
- net /PFC renamed PFC
- net /RST renamed RST
- net /SCR renamed SCR
- net /SPI_CLK renamed SPI_CLK
- net /SPI_MOSI renamed SPI_MOSI
- net /TCK renamed TCK
- net /TDI renamed TDI
- net /TDO renamed TDO
- net /THERM1 renamed THERM1
- net /THERM2 renamed THERM2
- net /TMS renamed TMS
- net /USART_RX renamed USART_RX
- net /USART_TX renamed USART_TX
- net /VAC_IN renamed Net-(J2-Pad10)
- net /VAC_SENSE renamed VAC_SENSE
- net /VBUS_IN renamed Net-(J2-Pad08)
- net /VBUS_SENSE renamed VBUS_SENSE
- net /VFAN_OUT renamed VFAN_OUT
- net /VREF renamed VREF
Routing:
- net VFAN_OUT: track 63.0 -> 75.6 mm, vias 1 -> 5
- net FAN_EN: track 19.2 -> 23.8 mm
- net CS_FAN: track 20.4 -> 24.2 mm
- net Net-(D14-K): track 16.0 -> 13.1 mm
- net Net-(D15-K): track 14.7 -> 17.0 mm
- net DRIVE_EN: track 51.9 -> 53.3 mm, vias 1 -> 3
- net SPI_MOSI: track 167.3 -> 167.9 mm
- net SPI_CLK: track 160.0 -> 160.6 mm

Commit message: changed pin assignments, improved hardware
Parts:
- removed C65, C90, C91, C92, C93, C94, C95: .1uf 885012208087, Capacitor_SMD:C_1206_3216Metric_Pad1.33x1.80mm_HandSolder
- removed C67, C68, C69, C70, C75, C76, C77, C78, C83, C84, C86, C87, C88: 2u2 C3225X7R1H225K250AB, Capacitor_SMD:C_1210_3225Metric_Pad1.33x2.70mm_HandSolder
- removed IC5: L4940D2T12-TR, Library:L4940D2T12-TR
- added C96: .1uf 885012208087, Capacitor_SMD:C_1206_3216Metric_Pad1.33x1.80mm_HandSolder, B.Cu at (40.0, 75.9)
- added D19: MBR0530, digikey-footprints:SOD-123, B.Cu at (46.8, 70.4)
- added D20: PMEG4050EP, Diode_SMD:D_SOD-128, B.Cu at (51.2, 31.0)
- added L1: 22u SRP7028A-220M, Library:INDPM7366X300N, B.Cu at (39.2, 36.8)
- added Q2: NTR5198NLT1G, Library:SOT96P237X111-3N, B.Cu at (31.3, 40.7)
- added R19: 1k MCU0805MD1051BP500, Resistor_SMD:R_0805_2012Metric_Pad1.20x1.40mm_HandSolder, B.Cu at (49.7, 74.9)
- added R20: 9k CRCW08059K10FKEAHP, Resistor_SMD:R_0805_2012Metric_Pad1.20x1.40mm_HandSolder, B.Cu at (47.7, 74.9)
- added R35: 10k CRCW080510K0DHEAP, Resistor_SMD:R_0805_2012Metric_Pad1.20x1.40mm_HandSolder, B.Cu at (32.2, 36.8)
- added R36: 150R KTR18EZPJ151, Resistor_SMD:R_1206_3216Metric_Pad1.30x1.75mm_HandSolder, F.Cu at (33.9, 54.2)
- added U11: AP1501A-12K5G-13, Package_TO_SOT_SMD:TO-263-5_TabPin3, B.Cu at (42.2, 22.7)
- C29: value 2u2 C3225X7R1H225K250AB -> 1n CGA3EAC0G2A102J080AA; footprint Capacitor_SMD:C_1210_3225Metric_Pad1.33x2.70mm_HandSolder -> Capacitor_SMD:C_0603_1608Metric_Pad1.08x0.95mm_HandSolder
- moved C29 32.8 mm to (30.5, 36.9), turned to 90 degrees
- moved C51 10.9 mm to (32.9, 21.6), turned to 90 degrees
- moved C64 7.90 mm to (30.5, 21.6), turned to 90 degrees
- moved C66 6.55 mm to (28.1, 21.6)
- moved L5 6.10 mm to (37.3, 45.1)
- moved C63 5.69 mm to (60.0, 64.1)
- moved C9 2.16 mm to (50.0, 61.3), turned to 180 degrees
- moved R10 1.41 mm to (34.4, 40.1)
- moved C52 0.90 mm to (50.5, 33.8)
- moved C82 0.60 mm to (45.0, 36.2)
- moved C38 0.20 mm to (49.5, 68.7)
- moved C58 0.20 mm to (57.2, 57.0)
Connections:
- net Net-(J2-Pad01) renamed I_L_IN
- net Net-(J2-Pad08) renamed VBUS_IN
- net Net-(J2-Pad10) renamed VAC_IN
- C29 pad 1: GND -> Net-(Q2-G)
- C29 pad 2: VFAN_OUT -> GND
- J1 pad 9: unconnected-(J1-Pad9) -> GND
- J10 pad 2: GND -> Net-(Q2-D)
- U1 pad 13: CT- -> INT
- U1 pad 15: CT+ -> LED_TMP
- U1 pad 16: LED_TMP -> LED_I_IN
- U1 pad 17: LED_I_IN -> 24V_SENSE
- U1 pad 2: GDT1_INA -> PMP_EN
- U1 pad 34: INT -> unconnected-(U1-PA12-Pad34)
- U1 pad 41: GDT2_INB -> unconnected-(U1-PB4-Pad41)
- U1 pad 42: GDT2_DIS -> GDT_B
- U1 pad 43: GDT2_INA -> GDT2_DIS
- U1 pad 46: GDT1_INB -> GDT_A
- U8 pad 1: GDT1_INA -> GDT_A
- U8 pad 2: GDT1_INB -> GDT_B
- U9 pad 1: GDT2_INA -> GDT_A
- U9 pad 2: GDT2_INB -> GDT_B
Routing:
- net GND: track 350.7 -> 293.2 mm, vias 111 -> 110
- net +24V: track 44.5 -> 80.2 mm, vias 19 -> 13
- net VDD: track 54.9 -> 23.3 mm, vias 21 -> 18
- net PMP_EN: track 0.00 -> 27.0 mm
- net GDT_B: track 0.00 -> 24.8 mm, vias 0 -> 2
- net GDT_A: track 0.00 -> 23.2 mm
- net Net-(Q2-G): track 0.00 -> 20.5 mm, vias 0 -> 1
- net 24V_SENSE: track 0.00 -> 19.5 mm, vias 0 -> 1
- net Net-(D20-K): track 0.00 -> 17.1 mm
- net GDT1_INB: track 15.8 -> 0.00 mm
- net GDT1_INA: track 15.5 -> 0.00 mm
- net INT: track 52.6 -> 40.2 mm, vias 2 -> 0
- net +12V: track 152.4 -> 140.9 mm
- net GDT2_INB: track 9.10 -> 0.00 mm
- net Net-(Q2-D): track 0.00 -> 7.89 mm, vias 0 -> 2
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
Commit message: ftdi board + random stuff
Parts:
- removed C85, C89: 2u2 C3225X7R1H225K250AB, Capacitor_SMD:C_1210_3225Metric_Pad1.33x2.70mm_HandSolder
- added C65: 150p VJ0603A151JXAAC, Capacitor_SMD:C_0603_1608Metric_Pad1.08x0.95mm_HandSolder, B.Cu at (27.6, 61.3)
- added C67: 150p VJ0603A151JXAAC, Capacitor_SMD:C_0603_1608Metric_Pad1.08x0.95mm_HandSolder, B.Cu at (24.3, 60.3)
- added C68: 10n VJ0603Y103KXJAC31X, Capacitor_SMD:C_0603_1608Metric_Pad1.08x0.95mm_HandSolder, B.Cu at (59.0, 63.2)
- added C69: 10n VJ0603Y103KXJAC31X, Capacitor_SMD:C_0603_1608Metric_Pad1.08x0.95mm_HandSolder, B.Cu at (59.1, 66.5)
- added C70: .1uf 885012208087, Capacitor_SMD:C_1206_3216Metric_Pad1.33x1.80mm_HandSolder, F.Cu at (35.1, 37.6)
- added D21: MBR0530, digikey-footprints:SOD-123, B.Cu at (31.2, 61.1)
- added J9: 3-647166-2, Library:36471662, F.Cu at (40.4, 60.5)
- added R37: 1k, Resistor_SMD:R_0805_2012Metric_Pad1.20x1.40mm_HandSolder, B.Cu at (63.3, 63.8)
- added U12: MCP9700Ax-ETT, Package_TO_SOT_SMD:SOT-23, F.Cu at (38.6, 35.5)
- C1, C11, C12, C14, C16, C17, C18, C19, C25, C36, C4, C56, C57, C58, C9, D2, D3, D4, D5, D6, D7, D8, R22, R29: moved to B.Cu
- IC3: value BD50FD0WHFP-TR -> LDL1117S50R; footprint Library:BD50FD0WHFPTR -> Library:SOT230P700X180-4N
- J8: value B4B-PH-SM4-TB -> 3-647166-2; footprint Library:CONN_B4B-PH-SM4-TB_JST -> Library:36471662
- R1, R17: value 3k CRCW08053K00FKTA -> 3k
- R10, R13, R21, R6, R8: value 1k MCU0805MD1051BP500 -> 1k; moved to B.Cu
- R11, R15: value 47k CRCW080547K0FKEA -> 47k
- R12, R16: value 470k CRCW0805470KFKTA -> 470k
- R14: value 5R1 ERJ-B1BF5R1U -> 2R2 35222R2JT; footprint Resistor_SMD:R_1020_2550Metric_Pad1.33x5.20mm_HandSolder -> Resistor_SMD:R_2512_6332Metric_Pad1.40x3.35mm_HandSolder; moved to B.Cu
- R18, R2: value 82k CRCW080582K0FKEA -> 82k
- R19, R3, R4, R7, R9: value 1k MCU0805MD1051BP500 -> 1k
- R20: value 9k CRCW08059K10FKEAHP -> 9k
- R33, R34, R35: value 10k CRCW080510K0DHEAP -> 10k
- R36: value 150R KTR18EZPJ151 -> 150R; footprint Resistor_SMD:R_1206_3216Metric_Pad1.30x1.75mm_HandSolder -> Resistor_SMD:R_0805_2012Metric_Pad1.20x1.40mm_HandSolder; moved to B.Cu
- R5: value 150R KTR18EZPJ151 -> 150R; footprint Resistor_SMD:R_1206_3216Metric_Pad1.30x1.75mm_HandSolder -> Resistor_SMD:R_0805_2012Metric_Pad1.20x1.40mm_HandSolder
- moved R10 25.0 mm to (42.8, 63.6), turned to 180 degrees
- moved C25 21.8 mm to (55.2, 66.7), turned to 0 degrees
- moved D2 21.4 mm to (42.6, 54.3)
- moved C6 21.3 mm to (38.5, 73.7), turned to -90 degrees
- moved C19 19.6 mm to (41.6, 50.6), turned to 0 degrees
- moved C17 19.4 mm to (47.4, 65.1)
- moved D8 18.5 mm to (48.4, 62.0)
- moved D13 17.8 mm to (33.6, 73.8), turned to 0 degrees
- moved D7 16.9 mm to (40.4, 54.3)
- moved R8 16.8 mm to (38.0, 50.8)
- moved C32 15.8 mm to (26.8, 79.5), turned to 180 degrees
- moved C33 15.3 mm to (26.8, 77.0), turned to 180 degrees
- moved R6 13.3 mm to (37.8, 84.2), turned to 90 degrees
- moved IC3 13.0 mm to (34.5, 66.7)
- moved C71 11.2 mm to (62.9, 28.7)
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Connections:
- IC3 pad 1: +24V -> GND
- IC3 pad 2: +24V -> +5V
- IC3 pad 3: GND -> +12V
- J8 pad 2: THERM1 -> THERM2
- U1 pad 26: MODE_IN -> THERM_BOARD
- U1 pad 34: unconnected-(U1-PA12-Pad34) -> MODE_IN
- U1 pad 41: unconnected-(U1-PB4-Pad41) -> JRST
Routing:
- net Net-(U12-V_{OUT}): track 0.00 -> 152.8 mm, vias 0 -> 2
- net VDD: track 23.3 -> 121.3 mm, vias 18 -> 15
- net VBUS_SENSE: track 109.4 -> 32.4 mm, vias 2 -> 1
- net +12V: track 140.9 -> 193.8 mm, vias 1 -> 5
- net I_L_IN: track 39.6 -> 68.2 mm, vias 0 -> 1
- net I_L: track 45.1 -> 20.9 mm, vias 2 -> 1
- net +24V: track 80.2 -> 102.2 mm, vias 13 -> 10
- net VBUS_IN: track 57.8 -> 75.0 mm, vias 0 -> 1
- net Net-(Q2-G): track 20.5 -> 10.1 mm, vias 1 -> 0
- net Net-(SW1-B): track 2.01 -> 11.9 mm
- net +5V: track 232.6 -> 242.0 mm, vias 5 -> 4
- net THERM_BOARD: track 0.00 -> 8.21 mm, vias 0 -> 1
- net INT: track 40.2 -> 33.9 mm, vias 0 -> 1
- net PFC: track 102.3 -> 107.6 mm
- net JRST: track 0.00 -> 5.32 mm
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- removed copper zone on B.Cu, net +5V
Other:
- board text added: "24V"
- board text added: "GDT 1"
- board text added: "GDT 2"
- board text added: "GND"
- board text added: "TH1"
- board text added: "TH2"
- board text removed: "THERM"
