File: hardware/booster-tc-driver/booster-tc-driver.kicad_pcb (KiCad board)
At the start: 4 copper layers, 53.3 x 72 mm, 174 parts, among them IC1 AD5160BRJZ5-RL7, IC2 AD5160BRJZ5-RL7, IC3 LDL1117S50R, IC4 CAT4109V-GT2, IC6 SI4564DY-T1-GE3, IC7 SI4564DY-T1-GE3, IC8 SI4564DY-T1-GE3, IC9 SI4564DY-T1-GE3, J1 62201021121, J10 3-647166-2, J2 EHT-105-01-S-D, J3 3-647166-2, J4 22-23-2021, J5 22-23-2021, J6 22-23-2021, J7 3-647166-2, J8 3-647166-2, J9 3-647166-2, Q1 T2N7002AK, Q2 NTR5198NLT1G, SW1 SW_SPDT, U1 STM32G474CBTx, U10 LT1963AxST-3.3, U11 AP1501A-12K5G-13, U12 MCP9700Ax-ETT, U2 AOZ1284PI, U3 CSTNE8M00G550000R0, U4 IF-D95T << must be T, U5 IF-E96E, U6 IF-D95T << must be T, U7 AOZ1284PI, U8 UCC21520DW, U9 UCC21520DW

Commit message: driver work
Parts:
- removed C24: .1uf 885012208087, Capacitor_SMD:C_1206_3216Metric_Pad1.33x1.80mm_HandSolder
- removed C46, C5: 2u2 C3225X7R1H225K250AB, Capacitor_SMD:C_1210_3225Metric_Pad1.33x2.70mm_HandSolder
- removed L4: 22u SRP7028A-220M, Library:INDPM7366X300N
- added L3: 22u IHLP3232DZER220M5A, Library:IND_IHLP-3232DZ_VIS-M, B.Cu at (52.9, 53.8)
- C68: value 10n VJ0603Y103KXJAC31X -> 1u C1206C105K5RACTU; footprint Capacitor_SMD:C_0603_1608Metric_Pad1.08x0.95mm_HandSolder -> Capacitor_SMD:C_1206_3216Metric_Pad1.33x1.80mm_HandSolder
- L1, L5: value 22u SRP7028A-220M -> 22u IHLP3232DZER220M5A; footprint Library:INDPM7366X300N -> Library:IND_IHLP-3232DZ_VIS-M
- L2: footprint Inductor_SMD:L_Murata_DFE201610P -> Library:LQM2MPN4R7NG0L
- moved C27 9.71 mm to (50.2, 42.0), turned to 0 degrees
- moved C19 7.45 mm to (35.2, 54.5)
- moved D2 6.65 mm to (36.2, 56.2), turned to 0 degrees
- moved R8 6.02 mm to (32.5, 53.2), turned to -90 degrees
- moved D7 5.75 mm to (36.2, 58.2), turned to 0 degrees
- moved C68 3.93 mm to (61.2, 60.0)
- moved R36 3.35 mm to (31.5, 48.8), turned to 180 degrees
- moved L5 3.10 mm to (38.5, 48.2)
- moved C58 2.03 mm to (62.5, 52.8)
- moved R11 1.80 mm to (46.8, 41.2), turned to -90 degrees
- moved C31 1.27 mm to (53.5, 41.6), turned to 90 degrees
- moved L1 1.22 mm to (39.0, 38.0)
- moved C12 1.15 mm to (59.0, 62.8)
- moved C81 1.15 mm to (45.0, 41.8)
- moved C20 0.50 mm to (36.8, 61.0)
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Connections:
- J10 pad 1: +12V -> Net-(Q2-D)
- J10 pad 2: Net-(Q2-D) -> +12V
- J8 pad 1: GND -> THERM2
- J8 pad 2: THERM2 -> GND
Routing:
- net GND: track 292.6 -> 273.8 mm
- net VFAN_OUT: track 67.9 -> 75.1 mm
- net Net-(Q2-G): track 10.1 -> 16.9 mm, vias 0 -> 2
- net +5V: track 242.0 -> 235.3 mm
- net Net-(D15-K): track 14.4 -> 20.2 mm
- net VBUS_SENSE: track 32.4 -> 37.6 mm
- net MODE_IN: track 70.5 -> 75.1 mm
- net VBUS_IN: track 75.0 -> 70.8 mm
- net FAN_EN: track 22.2 -> 25.1 mm
- net VDRIVE: track 92.3 -> 94.7 mm
- net CS_FAN: track 22.2 -> 24.4 mm
- net PMP_EN: track 27.4 -> 26.2 mm
- net +24V: track 102.2 -> 103.3 mm
- net VDD: track 121.3 -> 120.3 mm
- net DRIVE_EN: track 54.2 -> 53.5 mm
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