File: hardware/booster-tc-driver/booster-tc-driver.kicad_pcb (KiCad board)
At the start: 4 copper layers, 53.3 x 72 mm, 171 parts, among them IC1 AD5160BRJZ5-RL7, IC2 AD5160BRJZ5-RL7, IC3 LDL1117S50R, IC4 CAT4109V-GT2, IC6 SI4564DY-T1-GE3, IC7 SI4564DY-T1-GE3, IC8 SI4564DY-T1-GE3, IC9 SI4564DY-T1-GE3, J1 62201021121, J10 3-647166-2, J2 EHT-105-01-S-D, J3 3-647166-2, J4 22-23-2021, J5 22-23-2021, J6 22-23-2021, J7 3-647166-2, J8 3-647166-2, J9 3-647166-2, Q1 T2N7002AK, Q2 NTR5198NLT1G, SW1 SW_SPDT, U1 STM32G474CBTx, U10 LT1963AxST-3.3, U11 AP1501A-12K5G-13, U12 MCP9700Ax-ETT, U2 AOZ1284PI, U3 CSTNE8M00G550000R0, U4 IF-D95T << must be T, U5 IF-E96E, U6 IF-D95T << must be T, U7 AOZ1284PI, U8 UCC21520DW, U9 UCC21520DW

Commit message: v2 work
Parts:
- removed R22, R29: 5k CRCW06035K10FKEC, Resistor_SMD:R_0603_1608Metric_Pad0.98x0.95mm_HandSolder
- added JP1: SolderJumper_2_Open, Jumper:SolderJumper-2_P1.3mm_Open_RoundedPad1.0x1.5mm, F.Cu at (63.0, 56.5)
- added JP2: SolderJumper_2_Open, Jumper:SolderJumper-2_P1.3mm_Open_RoundedPad1.0x1.5mm, F.Cu at (51.1, 56.5)
- moved C2 0.30 mm to (41.0, 59.6)
- moved C20 0.30 mm to (36.5, 61.0)
Routing:
- net GND: track 273.8 -> 268.1 mm
- net +12V: track 193.2 -> 198.8 mm
- net Net-(U5-K): track 5.90 -> 10.0 mm
- net +5V: track 235.3 -> 237.9 mm
- net Net-(JP1-B): track 4.35 -> 5.45 mm
- net +24V: track 103.3 -> 104.1 mm
- net Net-(JP2-B): track 8.54 -> 8.00 mm
