File: hardware/booster-tc-driver/booster-tc-driver.kicad_sch (KiCad schematic)
At the start: 140 parts, among them IC1 AD5160BRJZ5-RL7, IC2 AD5160BRJZ5-RL7, IC3 LDL1117S50R, IC4 CAT4109V-GT2, J1 62201021121, J10 3-647166-2, J2 EHT-105-01-S-D, J3 3-647166-2, J6 22-23-2021, J7 3-647166-2, J8 3-647166-2, J9 3-647166-2, Q1 T2N7002AK, Q2 NTR5198NLT1G, SW1 SW_SPDT, U1 STM32G474CBTx, U10 LT1963AxST-3.3, U11 AP1501A-12K5G-13, U12 MCP9700Ax-ETT, U2 AOZ1284PI, U3 CSTNE8M00G550000R0, U4 IF-D95T << must be T, U5 IF-E96E, U6 IF-D95T << must be T, U7 AOZ1284PI

Commit message: driver work
Parts:
- removed C24: .1uf 885012208087, Capacitor_SMD:C_1206_3216Metric_Pad1.33x1.80mm_HandSolder, symbol Device:C
- removed C46, C5: 2u2 C3225X7R1H225K250AB, Capacitor_SMD:C_1210_3225Metric_Pad1.33x2.70mm_HandSolder, symbol Device:C
- removed L4: 22u SRP7028A-220M, Library:INDPM7366X300N, symbol Device:L
- added L3: 22u IHLP3232DZER220M5A, Library:IND_IHLP-3232DZ_VIS-M, symbol Device:L
- C68: value 10n VJ0603Y103KXJAC31X -> 1u C1206C105K5RACTU; footprint Capacitor_SMD:C_0603_1608Metric_Pad1.08x0.95mm_HandSolder -> Capacitor_SMD:C_1206_3216Metric_Pad1.33x1.80mm_HandSolder
- L1, L5: value 22u SRP7028A-220M -> 22u IHLP3232DZER220M5A; footprint Library:INDPM7366X300N -> Library:IND_IHLP-3232DZ_VIS-M
- L2: footprint Inductor_SMD:L_Murata_DFE201610P -> Library:LQM2MPN4R7NG0L
Connections:
- net +12V: now also J10.2; no longer J10.1
- net GND: now also J8.2; no longer J8.1
- net THERM2: now also J8.1; no longer J8.2
- net VFAN_OUT: now also L3.2
- net at Q2.3 (D): now also J10.1; no longer J10.2
- net at C23.2, D14.1 (K), U2.1 (LX): now also L3.1
Other:
- moved on the sheet: J10, J8
