File: hardware/booster-ftdi-board/booster-ftdi-board.kicad_sch (KiCad schematic)
At the start: 25 parts, among them J1 USB-B1HSB6, Q1 T2N7002AK, U1 FT231XS, U2 IF E96-E, U3 IF D95-T, U4 SN74LV1T34DBV, U5 SN74LV1T34DBV

Commit message: driver work
Changed lines of the file:
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@@
 		(dnp no)
 		(property "Reference" "R5"
-			(at 59.69 44.45 0)
+			(at 61.214 44.45 0)
 			(effects
 				(font
@@
 		)
 		(property "Value" "150R"
-			(at 59.69 46.99 0)
+			(at 61.214 46.99 0)
 			(effects
 				(font

Commit message: idk
Parts:
- J1: footprint Connector_USB:USB_B_OST_USB-B1HSxx_Horizontal -> Library:USB_B_OST_USB-B1HSxx_Horizontal
Changed lines of the file:
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@@
 			)
 		)
-		(property "Footprint" "Connector_USB:USB_B_OST_USB-B1HSxx_Horizontal"
+		(property "Footprint" "Library:USB_B_OST_USB-B1HSxx_Horizontal"
 			(at 29.21 86.36 0)
 			(effects

Commit message: v2 work
Parts:
- removed C10, C11, C4, C6, C7: 100n, Capacitor_SMD:C_0603_1608Metric, symbol Device:C
- removed C3: 47p, Capacitor_SMD:C_0603_1608Metric, symbol Device:C
- removed C5, C8, C9: 4u7, Capacitor_SMD:C_0603_1608Metric, symbol Device:C
- removed D1: 150060AS75000, LED_SMD:LED_0603_1608Metric, symbol Device:LED
- removed FB1: MI0805K400R-10, Resistor_SMD:R_0805_2012Metric, symbol Device:FerriteBead
- removed J1: USB-B1HSB6, Library:USB_B_OST_USB-B1HSxx_Horizontal, symbol Connector:USB_B
- removed Q1: T2N7002AK, Package_TO_SOT_SMD:SOT-23, symbol Transistor_FET:T2N7002AK
- removed R2: 27R, Resistor_SMD:R_0603_1608Metric, symbol Device:R
- removed R3: 1k, Resistor_SMD:R_0603_1608Metric, symbol Device:R
- removed R4, R5: 150R, Resistor_SMD:R_0603_1608Metric, symbol Device:R
- removed U1: FT231XS, Package_SO:SSOP-20_3.9x8.7mm_P0.635mm, symbol Interface_USB:FT231XS
- removed U2: IF E96-E, Library:IF-E96E, symbol New_Library:IF-E96E
- removed U3: IF D95-T, Library:IF-D95, symbol New_Library:IF-D95
- removed U4, U5: SN74LV1T34DBV, Package_TO_SOT_SMD:SOT-23-5, symbol Logic_LevelTranslator:SN74LV1T34DBV
- added C12: 100n, Capacitor_SMD:C_0805_2012Metric_Pad1.18x1.45mm_HandSolder, symbol Device:C
- added J2: UP2-AH-1-TH, digikey-footprints:USB_Male_A_UP2-AH-1-TH, symbol Connector:USB_A
- added R6: 150R, Resistor_SMD:R_0805_2012Metric_Pad1.20x1.40mm_HandSolder, symbol Device:R
- added U6: FT232RL, Package_SO:SSOP-28_5.3x10.2mm_P0.65mm, symbol Interface_USB:FT232RL
- added U7: IF E96-E, Library:IF-E96E, symbol New_Library:IF-E96E
- added U8: IF D95-T, Library:IF-D95, symbol New_Library:IF-D95
- C1: value 10n -> 4u7; footprint Capacitor_SMD:C_0603_1608Metric -> Capacitor_SMD:C_0805_2012Metric_Pad1.18x1.45mm_HandSolder
- C2: value 47p -> 100n; footprint Capacitor_SMD:C_0603_1608Metric -> Capacitor_SMD:C_0805_2012Metric_Pad1.18x1.45mm_HandSolder
- R1: value 27R -> 10k; footprint Resistor_SMD:R_0603_1608Metric -> Resistor_SMD:R_0805_2012Metric_Pad1.20x1.40mm_HandSolder
Connections:
- net USBI_N is gone; now on net GND: C2.1
- net USBI_P is gone; now on net VCC: R1.1
- net GND: now also C12.1, J2.4 (GND), U6.18 (GND), U6.21 (GND), U6.25 (AGND), U6.26 (TEST), U6.7 (GND), U8.1 (GND); no longer C2.2
- net VCC: now also C1.2, C2.2, J2.1 (VBUS), U6.20 (VCC), U6.4 (VCCIO), U7.2 (A), U8.3 (VCC)
- net USB_P: no longer names the net of R1.2
- net USB_P: now also U6.5 (RXD), U8.2 (OUT)
- new net: R6.1, U6.1 (TXD)
- new net: C12.2, U6.17 (3V3OUT)
- new net: R6.2, U7.1 (K)
- new net USB_+: J2.3 (D+), U6.15 (USBD+)
- new net USB_-: J2.2 (D-), U6.16 (USBD-)
- no-connect marks 10 -> 0
