File: hardware/booster-tc-driver-v2/booster-tc-driver.kicad_pcb (KiCad board)
At the start: 6 copper layers, 53.3 x 72 mm, 143 parts, among them IC1 CAT4109V-GT2, IC2 LDL1117S50R, IC3 AD5160BRJZ5-RL7, IC4 UCC27524AQDRQ1, IC5 UCC27524AQDRQ1, J1 62201021121, J10 22-23-2021, J2 EHT-105-01-S-D, J3 22-23-2021, J4 3-647166-2, J5 3-647166-2, J6 3-647166-2, J7 3-647166-2, J8 3-647166-2, J9 22-23-2021, Q1 T2N7002AK, SW1 SW_SPDT, U1 IF-D95T << must be T, U10 SQJ500AEP-T1_GE3, U11 SQJ500AEP-T1_GE3, U12 SQJ500AEP-T1_GE3, U13 SQJ500AEP-T1_GE3, U2 IF-E96E, U3 IF-D95T << must be T, U4 CSTNE8M00G550000R0, U5 STM32G474CBTx, U6 MCP9700Ax-ETT, U7 AP1501A-12K5G-13, U8 LT1963AxST-3.3, U9 AOZ1284PI

Commit message: driver v2 work
Parts:
- removed C13: 1n, Capacitor_SMD:C_0603_1608Metric_Pad1.08x0.95mm_HandSolder
- added L4: ACM7060-701-2PL-TL01, Library:IND_ACM7060_TDK, B.Cu at (29.2, 51.3)
- U4: moved to B.Cu
- moved D7 115.4 mm to (28.2, 80.2), turned to -90 degrees
- moved D8 114.6 mm to (27.0, 76.2), turned to 0 degrees
- moved D1 109.9 mm to (35.2, 58.0)
- moved C9 108.5 mm to (24.5, 70.2), turned to 0 degrees
- moved C10 108.3 mm to (24.5, 68.5), turned to 0 degrees
- moved C12 105.0 mm to (27.8, 74.2)
- moved C14 104.9 mm to (27.0, 71.0), turned to -90 degrees
- moved D9 104.2 mm to (34.2, 50.2), turned to -90 degrees
- moved C3 102.5 mm to (33.2, 71.5), turned to -90 degrees
- moved D10 101.9 mm to (36.8, 50.2), turned to 90 degrees
- moved C11 97.7 mm to (35.0, 70.1), turned to -90 degrees
- moved R10 90.8 mm to (25.2, 73.2), turned to -90 degrees
- moved C16 87.8 mm to (43.8, 72.5), turned to 0 degrees
- moved C17 87.6 mm to (43.8, 74.2)
- moved R9 84.8 mm to (31.8, 74.0), turned to 0 degrees
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Connections:
- J4 pad 1: CT+ -> Net-(J4-Pad1)
- J4 pad 2: CT- -> Net-(J4-Pad2)
Routing:
- net THERM2: track 1.40 -> 79.8 mm, vias 1 -> 3
- net SCR: track 3.10 -> 76.7 mm, vias 1 -> 3
- net THERM1: track 2.31 -> 70.1 mm, vias 1 -> 3
- net VAC_IN: track 2.00 -> 64.6 mm, vias 0 -> 2
- net PFC: track 4.04 -> 56.6 mm, vias 1 -> 2
- net I_L_IN: track 4.58 -> 48.1 mm, vias 0 -> 1
- net GND: track 189.2 -> 230.1 mm, vias 88 -> 97
- net VBUS_IN: track 1.50 -> 39.1 mm, vias 0 -> 1
- net VREF: track 1.37 -> 22.9 mm, vias 1 -> 3
- net VBUS_SENSE: track 2.24 -> 23.7 mm
- net I_L: track 2.07 -> 19.0 mm
- net VAC_SENSE: track 1.88 -> 17.9 mm
- net VFAN_OUT: track 38.5 -> 52.3 mm, vias 1 -> 3
- net +12V: track 51.3 -> 60.0 mm, vias 2 -> 4
- net VDDA: track 1.46 -> 10.1 mm
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
Commit message: pcb work
Parts:
- removed J1: 62201021121, Library:CONN_62201021121_WRE
- added G***: LOGO, Library:tclogo, F.Cu at (39.0, 50.8)
- added J11: 3220-10-0300-00, Library:CNC_3220-10-0300-00, F.Cu at (44.0, 62.5)
Routing:
- net TMS: track 21.9 -> 7.46 mm, vias 1 -> 0
- net TCK: track 22.9 -> 11.0 mm, vias 1 -> 0
- net TDO: track 25.4 -> 13.8 mm, vias 1 -> 0
- net RST: track 34.3 -> 22.8 mm, vias 1 -> 0
- net TDI: track 26.0 -> 17.3 mm, vias 1 -> 0
- net GND: track 230.1 -> 236.7 mm
- net THERM2: track 79.8 -> 74.6 mm
- net MODE_IN: track 27.5 -> 23.9 mm
- net THERM1: track 70.1 -> 66.9 mm
- net VDD: track 49.9 -> 50.9 mm, vias 13 -> 14
- net Net-(J4-Pad1): track 3.51 -> 4.20 mm
Other:
- board text added: "- +24"
- board text added: "CT"
- board text added: "FAN"
- board text added: "GDT1"
- board text added: "GDT2"
- board text added: "PFC"
- board text added: "PMP"
- board text added: "PROG"
- board text added: "TH1"
- board text added: "TH2"
