File: hardware/booster-tc-driver-v2/booster-tc-driver.kicad_sch (KiCad schematic)
At the start: 115 parts, among them IC1 CAT4109V-GT2, IC2 LDL1117S50R, IC3 AD5160BRJZ5-RL7, J1 62201021121, J2 EHT-105-01-S-D, J3 22-23-2021, J4 3-647166-2, J5 3-647166-2, J6 3-647166-2, J7 3-647166-2, J8 3-647166-2, Q1 T2N7002AK, SW1 SW_SPDT, U1 IF-D95T << must be T, U2 IF-E96E, U3 IF-D95T << must be T, U4 CSTNE8M00G550000R0, U5 STM32G474CBTx, U6 MCP9700Ax-ETT, U7 AP1501A-12K5G-13, U8 LT1963AxST-3.3, U9 AOZ1284PI

Commit message: driver v2 work
Parts:
- removed C13: 1n, Capacitor_SMD:C_0603_1608Metric_Pad1.08x0.95mm_HandSolder, symbol Device:C
- added L4: ACM7060-701-2PL-TL01, Library:IND_ACM7060_TDK, symbol New_Library:ACM7060-701-2PL-TL01
Connections:
- net CT+: now also L4.2; no longer J4.1
- net CT-: now also L4.1; no longer J4.2
- new net: J4.2, L4.3
- new net: J4.1, L4.4
Other:
- moved on the sheet: C11, D11, IC1, J4, R12, R13, R14

Commit message: pcb work
Parts:
- removed J1: 62201021121, Library:CONN_62201021121_WRE, symbol 2024-07-01_18-43-42:62201021121
- added J11: 3220-10-0300-00, Library:CNC_3220-10-0300-00, symbol dk_Rectangular-Connectors-Headers-Male-Pins:3220-10-0100-00
Connections:
- net GND: now also J11.3, J11.5, J11.9
- net RST: now also J11.10
- net TCK: now also J11.4
- net TDI: now also J11.8
- net TDO: now also J11.6
- net TMS: now also J11.2
- net VDD: now also J11.1
