File: hardware/booster-pfc-v3/booster-tc.kicad_pcb (KiCad board)
At the start: 2 copper layers, 108 x 114.3 mm, 71 parts, among them J10 74650074R, J12 74650074R, J13 74650074R, J14 61201021621, J2 74650074R, J3 74650074R, J4 74650074R, Q3 DMN6075S, Q4 IPW60R016CM8, T2 78601/1JC-R, U3 MGJ2D241505SC, U5 STGAP2SM, U6 ACS770LCB-100U-PFF-T, U7 MCP6L02T-E/SN

Commit message: pfc v3
Parts:
- removed C27, C35: 1u, Library:B32672P4105K000
- removed U7: MCP6L02T-E/SN, Package_SO:MSOP-8_3x3mm_P0.65mm
- added C12: 0.1u, Capacitor_SMD:C_0805_2012Metric, F.Cu at (145.0, 127.8)
- added C16: 0.1u, Capacitor_SMD:C_0805_2012Metric, F.Cu at (108.5, 133.8)
- added H1: MountingHole, MountingHole:MountingHole_3.2mm_M3, F.Cu at (154.5, 53.5)
- added H2: MountingHole, MountingHole:MountingHole_3.2mm_M3, F.Cu at (53.5, 53.5)
- added H3: MountingHole, MountingHole:MountingHole_3.2mm_M3, F.Cu at (154.5, 160.8)
- added H4: MountingHole, MountingHole:MountingHole_3.2mm_M3, F.Cu at (53.5, 160.8)
- added U1: MCP6L02T-E/SN, Package_SO:SOIC-8_3.9x4.9mm_P1.27mm, F.Cu at (110.2, 156.6)
- moved D4 201.9 mm to (52.9, 154.2)
- moved D3 191.9 mm to (71.5, 149.2), turned to -90 degrees
- moved C2 190.4 mm to (68.0, 158.5), turned to -90 degrees
- moved R15 187.0 mm to (52.8, 150.8), turned to 180 degrees
- moved R18 185.9 mm to (52.8, 147.5), turned to 180 degrees
- moved Q1 183.8 mm to (75.0, 149.5), turned to 180 degrees
- moved D2 182.9 mm to (71.5, 152.5), turned to 90 degrees
- moved T1 179.8 mm to (62.0, 151.0), turned to 180 degrees
- moved C5 178.8 mm to (78.6, 149.5), turned to 90 degrees
- moved D9 169.4 mm to (76.5, 120.5), turned to 90 degrees
- moved C7 168.7 mm to (100.0, 158.5), turned to 90 degrees
- moved C10 165.5 mm to (102.5, 158.5), turned to 90 degrees
- moved R8 164.1 mm to (74.8, 152.8), turned to 180 degrees
- moved C14 161.4 mm to (105.0, 154.6), turned to -90 degrees
- moved R26 160.6 mm to (81.9, 145.2)
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- renumbered C38 to C1, C43 to C10, C29 to C11, C41 to C13, C44 to C14, C26 to C15, C31 to C17, C36 to C18, C32 to C19, C24 to C2, C37 to C20, C33 to C21, C34 to C22, C30 to C3, C25 to C4, C13 to C5, C39 to C6, C42 to C7, C28 to C8, C40 to C9, D16 to D1, D14 to D2, D13 to D3, D12 to D4, D7 to D5, D10 to D6, D9 to D7, D11 to D8, D15 to D9, J2 to J1, J3 to J2, J4 to J3, J10 to J4, J14 to J5, J13 to J6, J12 to J7, Q3 to Q1, Q4 to Q2, R21 to R1, R30 to R10, R38 to R11, R39 to R12, R31 to R13, R40 to R14, R18 to R15, R32 to R16, R41 to R17, R20 to R18, R23 to R19, R43 to R2, R24 to R20, R33 to R21, R42 to R22, R25 to R23, R26 to R24, R27 to R25, R28 to R26, R44 to R3, R34 to R4, R35 to R5, R36 to R6, R37 to R7, R22 to R8, R29 to R9, T2 to T1, U3 to U2, U5 to U3, U6 to U4
Routing:
- net +5V: track 0.00 -> 159.6 mm, vias 0 -> 3
- net Net-(D5-G): track 0.00 -> 132.5 mm, vias 0 -> 1
- net Net-(D7-G): track 0.00 -> 101.4 mm, vias 0 -> 1
- net /L+: track 0.00 -> 95.1 mm, vias 0 -> 1
- net VBUS_SENSE: track 0.00 -> 84.7 mm, vias 0 -> 1
- net SCR_TRIG: track 0.00 -> 82.7 mm, vias 0 -> 1
- net AC2: track 0.00 -> 82.4 mm, vias 0 -> 1
- net VAC_SENSE: track 0.00 -> 80.4 mm, vias 0 -> 1
- net AC1: track 0.00 -> 80.3 mm, vias 0 -> 1
- net GND: track 0.00 -> 78.2 mm, vias 0 -> 8
- net V+: track 0.00 -> 58.0 mm, vias 0 -> 1
- net ISENSE: track 0.00 -> 44.1 mm
- net +24V: track 0.00 -> 31.2 mm
- net Net-(U1A-+): track 0.00 -> 24.6 mm
- net FET_GATE: track 0.00 -> 23.5 mm, vias 0 -> 1
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- added copper zone on B.Cu, net /L+
- added copper zone on B.Cu, net /LSW
- added copper zone on B.Cu, net /SW
- added copper zone on F.Cu, net /SW
- added copper zone on B.Cu, net AC1
- added copper zone on F.Cu, net AC2
- added copper zone on In1.Cu, net GND
- added copper zone on F.Cu, net V+
- added copper zone on B.Cu, net V-
Other:
- board size 108 x 114.3 mm -> 108 x 114.2 mm
- copper layers 2 -> 4
- board text added: "+"
- board text added: "-"
- board text added: "L"
- board text added: "~"

Commit message: pfc v3 finalized
Parts:
- moved D1 14.6 mm to (100.8, 137.8)
- moved C2 14.3 mm to (82.2, 159.7)
- moved C4 14.3 mm to (87.8, 157.9)
- moved C5 14.3 mm to (92.8, 150.7)
- moved D2 14.3 mm to (85.7, 153.7)
- moved D3 14.3 mm to (85.7, 150.4)
- moved Q1 14.3 mm to (89.2, 150.7)
- moved R1 14.3 mm to (95.3, 150.7)
- moved R15 14.3 mm to (67.0, 151.9)
- moved R18 14.3 mm to (67.0, 148.7)
- moved R8 14.3 mm to (89.0, 153.9)
- moved T1 14.3 mm to (76.2, 152.2)
- moved D4 14.3 mm to (67.1, 155.4)
- moved R25 13.0 mm to (94.8, 136.0)
- moved R26 13.0 mm to (91.0, 136.0)
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Routing:
- net AC2: track 82.4 -> 64.8 mm
- net AC1: track 80.3 -> 63.0 mm
- net +5V: track 159.6 -> 144.8 mm
- net SCR_TRIG: track 82.7 -> 68.4 mm
- net /L+: track 95.1 -> 81.3 mm
- net Net-(D5-G): track 132.5 -> 118.8 mm
- net Net-(D7-G): track 101.4 -> 87.6 mm
- net Net-(U1A-+): track 24.6 -> 17.2 mm
- net Net-(R24-Pad1): track 1.92 -> 8.84 mm
- net GND: track 78.2 -> 71.4 mm
- net Net-(D1--): track 11.9 -> 5.83 mm
- net V+: track 58.0 -> 62.8 mm
- net Net-(D1-+): track 9.75 -> 5.83 mm
- net V-: track 8.52 -> 6.48 mm
- net Net-(U1A--): track 16.6 -> 14.6 mm

Commit message: idk
Parts:
- added C23: 0.1u, Capacitor_SMD:C_0805_2012Metric, F.Cu at (130.0, 141.7)
- added C24: 0.1u, Capacitor_SMD:C_0805_2012Metric, F.Cu at (130.0, 145.5)
Routing:
- net V-: track 6.48 -> 20.6 mm, vias 2 -> 3
- net Net-(U2-+VOUT): track 22.4 -> 26.7 mm, vias 0 -> 1
- net Net-(U2--VOUT): track 22.1 -> 26.3 mm
Other:
- outline, holes or cut-outs redrawn
