File: hardware/booster-pfc-v3/booster-tc.kicad_sch (KiCad schematic)
At the start: 71 parts, among them J10 74650074R, J12 74650074R, J13 74650074R, J14 61201021621, J2 74650074R, J3 74650074R, J4 74650074R, Q3 DMN6075S, Q4 IPW60R016CM8, T2 78601/1JC-R, U3 MGJ2D241505SC, U5 STGAP2SM, U6 ACS770LCB-100U-PFF-T, U7 MCP6L02T-E/SN

Commit message: pfc v3
Parts:
- removed C27, C35: 1u, Library:B32672P4105K000, symbol Device:C
- removed U7: MCP6L02T-E/SN, Package_SO:MSOP-8_3x3mm_P0.65mm, symbol Amplifier_Operational:MCP6L02x-xSN
- added C12, C16: 0.1u, Capacitor_SMD:C_0805_2012Metric, symbol Device:C
- added H1, H2, H3, H4: MountingHole, MountingHole:MountingHole_3.2mm_M3, symbol Mechanical:MountingHole
- added U1: MCP6L02T-E/SN, Package_SO:SOIC-8_3.9x4.9mm_P1.27mm, symbol Amplifier_Operational:MCP6L02x-xSN
- renumbered C38 to C1, C43 to C10, C29 to C11, C41 to C13, C44 to C14, C26 to C15, C31 to C17, C36 to C18, C32 to C19, C24 to C2, C37 to C20, C33 to C21, C34 to C22, C30 to C3, C25 to C4, C13 to C5, C39 to C6, C42 to C7, C28 to C8, C40 to C9, D16 to D1, D14 to D2, D13 to D3, D12 to D4, D7 to D5, D10 to D6, D9 to D7, D11 to D8, D15 to D9, J2 to J1, J3 to J2, J4 to J3, J10 to J4, J14 to J5, J13 to J6, J12 to J7, Q3 to Q1, Q4 to Q2, R21 to R1, R30 to R10, R38 to R11, R39 to R12, R31 to R13, R40 to R14, R18 to R15, R32 to R16, R41 to R17, R20 to R18, R23 to R19, R43 to R2, R24 to R20, R33 to R21, R42 to R22, R25 to R23, R26 to R24, R27 to R25, R28 to R26, R44 to R3, R34 to R4, R35 to R5, R36 to R6, R37 to R7, R22 to R8, R29 to R9, T2 to T1, U3 to U2, U5 to U3, U6 to U4
Connections:
- net +5V: now also C12.2, C16.2, U1.8 (V+)
- net GND: now also C12.1, C16.1, U1.4 (V-)
- net VAC_SENSE: now also U1.1
- net VBUS_SENSE: now also U1.7
- net at C14.2, C7.2, R12.2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: now also U1.2 (-)
- net at C10.1, C7.1, R11.2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: now also U1.3 (+)
- net at C6.1, C9.1, R13.1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: now also U1.5 (+)
- net at C13.2, C6.2, R10.2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: now also U1.6 (-)

Commit message: pfc v3 finalized
Other:
- moved on the sheet: C12
Changed lines of the file:
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@@
 	(wire
 		(pts
-			(xy 96.52 95.25) (xy 97.79 95.25)
+			(xy 95.25 95.25) (xy 96.52 95.25)
 		)
 		(stroke
@@
 	(wire
 		(pts
+			(xy 104.14 95.25) (xy 105.41 95.25)
+		)
+		(stroke
+			(width 0)
+			(type default)
+		)
+	)
+	(wire
+		(pts
 			(xy 162.56 29.21) (xy 162.56 39.37)
 		)
@@
 	(symbol
 		(lib_id "Device:C")
-		(at 101.6 95.25 90)
+		(at 100.33 95.25 90)
 		(unit 1)
 		(exclude_from_sim no)
@@
 		(dnp no)
 		(property "Reference" "C12"
-			(at 99.06 91.44 90)
+			(at 97.79 91.44 90)
 			(effects
 				(font
@@
 		)
 		(property "Value" "0.1u"
-			(at 100.33 93.98 90)
+			(at 99.06 93.98 90)
 			(effects
 				(font
@@
 		)
 		(property "Footprint" "Capacitor_SMD:C_0805_2012Metric"
-			(at 105.41 94.2848 0)
+			(at 104.14 94.2848 0)
 			(effects
 				(font
@@
 		)
 		(property "Datasheet" "~"
-			(at 101.6 95.25 0)
+			(at 100.33 95.25 0)
 			(effects
 				(font
@@
 		)
 		(property "Description" "Unpolarized capacitor"
-			(at 101.6 95.25 0)
+			(at 100.33 95.25 0)
 			(effects
 				(font
@@
 	(symbol
 		(lib_id "power:GND")
-		(at 96.52 95.25 270)
+		(at 95.25 95.25 270)
 		(unit 1)
 		(exclude_from_sim no)
@@
 		(dnp no)
 		(property "Reference" "#PWR010"
-			(at 90.17 95.25 0)
+			(at 88.9 95.25 0)
 			(effects
 				(font
@@
 		)
 		(property "Value" "GND"
-			(at 92.71 95.25 0)
+			(at 91.44 95.25 0)
 			(effects
 				(font
@@
 		)
 		(property "Footprint" ""
-			(at 96.52 95.25 0)
+			(at 95.25 95.25 0)
 			(effects
 				(font
@@
 		)
 		(property "Datasheet" ""
-			(at 96.52 95.25 0)
+			(at 95.25 95.25 0)
 			(effects
 				(font
@@
 		)
 		(property "Description" "Power symbol creates a global label with name \"GND\" , ground"
-			(at 96.52 95.25 0)
+			(at 95.25 95.25 0)
 			(effects
 				(font

Commit message: idk
Parts:
- added C23, C24: 0.1u, Capacitor_SMD:C_0805_2012Metric, symbol Device:C
Connections:
- net V-: now also C23.2, C24.1
- net at C11.1, C8.1, U2.7 (+VOUT)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: now also C23.1
- net at C11.2, C8.2, U2.5 (-VOUT)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: now also C24.2
